File: Electronica/V2/V2.kicad_pcb (KiCad board)
At the start: 2 copper layers, 69.3 x 46.2 mm, 20 parts, among them J5 On/Off General

Commit message: placa v2 con xt30
Parts:
- Bateria: renamed from BATERIA; footprint Connector_Molex:Molex_KK-254_AE-6410-02A_1x02_P2.54mm_Vertical -> Connector_AMASS:AMASS_XT30U-F_1x02_P5.0mm_Vertical
- moved Bateria 5.09 mm to (91.0, 72.3)
- renumbered ADS1115 to ASD1115
Routing:
- net GND: track 283.8 -> 288.8 mm
- net Net-(D1-A): track 5.00 -> 8.03 mm
