File: Electronica/V2/V2.kicad_sch (KiCad schematic)
At the start: 20 parts, among them J1 Conn_01x03_Pin, J2 Power Input 1, J3 Conn_01x05_Pin, J4 Conn_01x03_Pin, J5 On/Off General, J6 Conn_01x05_Pin, J7 Conn_01x05_Pin, J8 Conn_01x05_Pin, J9 Conn_01x05_Pin, SW1 SW_DIP_x04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

Commit message: placa v2 con xt30
Parts:
- J2: footprint Connector_Molex:Molex_KK-254_AE-6410-02A_1x02_P2.54mm_Vertical -> Connector_AMASS:AMASS_XT30U-F_1x02_P5.0mm_Vertical
Changed lines of the file:
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@@
 			)
 		)
-		(property "Footprint" "Connector_Molex:Molex_KK-254_AE-6410-02A_1x02_P2.54mm_Vertical"
+		(property "Footprint" "Connector_AMASS:AMASS_XT30U-F_1x02_P5.0mm_Vertical"
 			(at 22.86 76.2 0)
 			(effects
